File: LPDataLogger/KiCadProjectFiles/LPDataLogger.kicad_pcb (KiCad board)
At the start: 2 copper layers, 22 parts, among them J1 Micro_SD_Card_Det2, J2 Conn_01x04, J3 JST BM03B-GHS-TBT, J4 JST B2P-VH-FB-B, U1 MCP96L00T-E_MX, U2 Pico 2, U3 FSM300

Commit message: Finished V1 of the low power data logger
Parts:
- removed the R3 at (72.5, 68.9)
- removed the R4 at (72.5, 71.4)
- added H1: MountingHole_Pad, MountingHole:MountingHole_3.5mm_Pad, F.Cu at (129.0, 110.5)
- added H2: MountingHole_Pad, MountingHole:MountingHole_3.5mm_Pad, F.Cu at (129.0, 118.6)
- H3, H4, H5, H6: footprint MountingHole:MountingHole_2.7mm_M2.5_Pad -> LPDataLogger:MountingHole_2.7mm_M2.5_Pad_with_stencil_hole
- TP1: footprint Connector_PinHeader_2.54mm:PinHeader_1x04_P2.54mm_Vertical -> Connector_PinHeader_2.54mm:PinHeader_2x02_P2.54mm_Vertical
- U1: footprint Package_DFN_QFN:QFN-20-1EP_5x5mm_P0.65mm_EP3.35x3.35mm_ThermalVias -> Package_DFN_QFN:QFN-20-1EP_5x5mm_P0.65mm_EP3.35x3.35mm
- moved H5 131.0 mm to (185.4, 128.3)
- moved U2 119.9 mm to (167.6, 104.1)
- moved H6 118.6 mm to (185.4, 82.5)
- moved J4 111.4 mm to (184.6, 96.5), turned to 90 degrees
- moved J3 103.3 mm to (184.4, 104.9), turned to -90 degrees
- moved H3 93.7 mm to (129.5, 128.3)
- moved C2 91.2 mm to (143.9, 115.6), turned to 180 degrees
- moved C1 87.8 mm to (139.2, 113.5), turned to -90 degrees
- moved U3 85.6 mm to (144.3, 91.7)
- moved J1 83.7 mm to (148.8, 123.2), turned to 180 degrees
- moved R2 81.6 mm to (135.6, 118.1)
- moved R1 78.2 mm to (135.6, 110.0)
- moved R3 76.4 mm to (141.2, 107.4), turned to -90 degrees
- moved R4 73.5 mm to (139.2, 107.4), turned to -90 degrees
- moved JP1 71.3 mm to (151.9, 106.9)
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- renumbered R5 to R3, R6 to R4
Connections:
- U1 pad 16: Net-(U1-ADDR) -> GND
Routing:
- net /I2C_SDA: track 0.00 -> 50.4 mm, vias 0 -> 2
- net /I2C_SCL: track 0.00 -> 44.1 mm, vias 0 -> 2
- net /FSM300_RESET: track 0.00 -> 28.9 mm
- net /HINTN: track 0.00 -> 27.4 mm
- net Net-(JP1-C): track 0.00 -> 26.4 mm, vias 0 -> 2
- net /UART_MAIN_TO_LOGGER: track 0.00 -> 25.0 mm
- net /UART_LOGGER_TO_MAIN: track 0.00 -> 24.4 mm
- net /SD_SPI_CLK: track 0.00 -> 22.7 mm
- net /SD_SPI_MISO: track 0.00 -> 18.6 mm, vias 0 -> 1
- net /SD_SPI_MOSI: track 0.00 -> 17.6 mm
- net +3V3: track 0.00 -> 14.6 mm, vias 0 -> 5
- net +BATT: track 0.00 -> 13.9 mm
- net /SD_SPI_CS: track 0.00 -> 13.4 mm
- net Net-(U1-VIN-): track 0.00 -> 9.89 mm
- net Net-(U1-VIN+): track 0.00 -> 8.70 mm
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- added copper zone on In2.Cu, net +3V3
- added copper zone on B.Cu, net GND
- added copper zone on F.Cu, net GND
- added copper zone on In1.Cu, net GND
Other:
- board outline added: 66 x 55.9 mm
- copper layers 2 -> 4
- board text added: "+"
- board text added: "+1.8V to +5.5V"
- board text added: "-"
- board text added: "3v3"
- board text added: "BOOTN | 3V3"
- board text added: "GND"
- board text added: "KRUPS Low Power Data Logger 04-10-2025 V1 | Serial Number:"
- board text added: "PS1 | GND"
- board text added: "Space Systems Lab University of Kentucky Lexington KY, USA, Earth"

Commit message: added silkscreen, schematic labels for UART pins
Other:
- board text added: "TXD RXD GND"
Changed lines of the file:
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@@
 		(tags "connector JST GH vertical")
 		(property "Reference" "J3"
-			(at 0 -4 90)
+			(at -3.61 2.794 90)
 			(layer "F.SilkS")
 			(effects
@@
 			)
 			(justify left bottom)
+		)
+	)
+	(gr_text "TXD\nRXD\nGND"
+		(at 187.325 107.315 0)
+		(layer "F.SilkS")
+		(effects
+			(font
+				(size 1 1)
+				(thickness 0.127)
+			)
+			(justify left bottom)
