File: LPDataLogger/KiCadProjectFiles/LPDataLogger.kicad_sch (KiCad schematic)
At the start: 24 parts, among them J1 Micro_SD_Card_Det2, J2 Conn_01x04, J3 JST BM03B-GHS-TBT, J4 JST B2P-VH-FB-B, U1 MCP96L00T-E_MX, U2 Pico 2, U3 FSM300

Commit message: Finished V1 of the low power data logger
Parts:
- removed R3: 10k, Resistor_SMD:R_0603_1608Metric_Pad0.98x0.95mm_HandSolder, symbol Device:R
- removed R4: 4.3k, Resistor_SMD:R_0603_1608Metric_Pad0.98x0.95mm_HandSolder, symbol Device:R
- H1, H2: footprint KRUPS_Footprints:2,8-PAD -> MountingHole:MountingHole_3.5mm_Pad; now left out of the parts list
- H3, H4, H5, H6: footprint MountingHole:MountingHole_2.7mm_M2.5_Pad -> LPDataLogger:MountingHole_2.7mm_M2.5_Pad_with_stencil_hole
- J2: now left out of the parts list
- J3: Digikey Part Number (none) -> 455-BM03B-GHS-TBTCT-ND
- J4: Digikey Part Number (none) -> 455-B2P-VH-FB-B-ND
- R3: renamed from R5; Digikey Part Number (none) -> 13-RC0603FR-1310KLTR-ND
- R4: renamed from R6; Digikey Part Number (none) -> 13-RC0603FR-1310KLTR-ND
- TP1: footprint Connector_PinHeader_2.54mm:PinHeader_1x04_P2.54mm_Vertical -> Connector_PinHeader_2.54mm:PinHeader_2x02_P2.54mm_Vertical; now left out of the parts list
- U1: footprint Package_DFN_QFN:QFN-20-1EP_5x5mm_P0.65mm_EP3.35x3.35mm_ThermalVias -> Package_DFN_QFN:QFN-20-1EP_5x5mm_P0.65mm_EP3.35x3.35mm
- U2: Digikey Part Number (none) -> 2648-SC1631CT-ND
Connections:
- net GND: now also U1.16 (ADDR)
Other:
- note added: "Raspberry Pi Pico 2 4MB flash"

Commit message: added silkscreen, schematic labels for UART pins
Other:
- note added: "RXD"
- note added: "TXD"
Changed lines of the file:
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@@
+		)
+	)
+	(text "RXD"
+		(exclude_from_sim no)
+		(at 17.018 56.388 0)
+		(effects
+			(font
+				(size 1.27 1.27)
+			)
 		)
 	)
@@
 		)
 	)
+	(text "TXD"
+		(exclude_from_sim no)
+		(at 17.018 49.022 0)
+		(effects
+			(font
+				(size 1.27 1.27)
+			)
+		)
+	)

Commit message: fixed LPDL BOM
Parts:
- C1, C2, C3: Digikey Part Number 0603B104K500XD -> 311-1088-1-ND
- J1: Digikey Part Number WM6357TR-ND -> WM6357CT-ND
- R1, R2: Digikey Part Number 311-100GRTR-ND -> 311-100GRCT-ND
- R3, R4: Digikey Part Number 13-RC0603FR-1310KLTR-ND -> 13-RC0603FR-1310KLCT-ND
- U1: Digikey Part Number MCP96L00T-E/MXTR-ND -> MCP96L00T-E/MXCT-ND
Changed lines of the file:
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@@
 			)
 		)
-		(property "Digikey Part Number" "WM6357TR-ND"
+		(property "Digikey Part Number" "WM6357CT-ND"
 			(at 250.19 43.18 0)
 			(effects
@@
 			)
 		)
-		(property "Digikey Part Number" "311-100GRTR-ND"
+		(property "Digikey Part Number" "311-100GRCT-ND"
 			(at 116.84 30.48 0)
 			(effects
@@
 			)
 		)
-		(property "Digikey Part Number" "0603B104K500XD"
+		(property "Digikey Part Number" "311-1088-1-ND"
 			(at 128.27 27.94 0)
 			(effects
@@
 			)
 		)
-		(property "Digikey Part Number" "MCP96L00T-E/MXTR-ND"
+		(property "Digikey Part Number" "MCP96L00T-E/MXCT-ND"
 			(at 156.21 34.29 0)
 			(effects
@@
 			)
 		)
-		(property "Digikey Part Number" "13-RC0603FR-1310KLTR-ND"
+		(property "Digikey Part Number" "13-RC0603FR-1310KLCT-ND"
 			(at 261.62 82.55 0)
 			(effects
@@
 			)
 		)
-		(property "Digikey Part Number" "13-RC0603FR-1310KLTR-ND"
+		(property "Digikey Part Number" "13-RC0603FR-1310KLCT-ND"
 			(at 261.62 80.01 0)
 			(effects
@@
 			)
 		)
-		(property "Digikey Part Number" "0603B104K500XD"
+		(property "Digikey Part Number" "311-1088-1-ND"
 			(at 177.8 30.48 0)
 			(effects
@@
 			)
 		)
-		(property "Digikey Part Number" "0603B104K500XD"
+		(property "Digikey Part Number" "311-1088-1-ND"
 			(at 111.76 71.12 0)
 			(effects
@@
 			)
 		)
-		(property "Digikey Part Number" "311-100GRTR-ND"
+		(property "Digikey Part Number" "311-100GRCT-ND"
 			(at 116.84 25.4 0)
 			(effects
